File: SAR_pcb_v2A/SAR_pcb.kicad_pcb (KiCad board)
At the start: 4 copper layers, 67.6 x 49.5 mm, 33 parts, among them J1 Conn_Coaxial_Power, J10 Conn_Coaxial, J2 Conn_Coaxial_Power, J3 Conn_02x10_Top_Bottom, J4 Conn_01x06, J9 Conn_Coaxial, SW1 SW_Push, U2 10B_SAR

Commit message: digikey car
Routing:
- added copper zone on PWR, net VDD
- added copper zone on PWR, net VDDPST
- added copper zone on PWR, net VREF
- removed copper zone on VDD, net VDD
- removed copper zone on VDD, net VDDPST
- removed copper zone on VDD, net VREF
